File: hardware/numpad/numpad/powerreg.kicad_sch (KiCad schematic)
At the start: 0 parts

Commit message: connectors for other modules
Other:
- note added: "Power Regulation. Buck Converter 5v to 3.3v"
- note removed: "Power Regulation. Pretty Straight Forward. Buck Converter 5v to 3.3v"
Changed lines of the file:
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@@
 	(generator_version "9.0")
 	(paper "A4")
-	(text "Power Regulation. Pretty Straight Forward.\nBuck Converter 5v to 3.3v\n"
+	(text "Power Regulation.\nBuck Converter 5v to 3.3v\n"
 		(exclude_from_sim no)
 		(at 97.79 99.568 0)
