File: hardware/numpad/numpad/matrixrot.kicad_sch (KiCad schematic)
At the start: 56 parts, among them SW1 ROT_SKYLOONG_HS

Commit message: progreers
Parts:
- added D29: 1N4148, PCM_Diode_THT_AKL:D_DO-35_SOD27_P7.62mm_Horizontal, symbol PCM_Diode_AKL:1N4148
- renumbered MX1 to MACRO_A1, MX2 to MACRO_B1, MX3 to MACRO_C1, MX4 to MACRO_D1, MX22 to MACRO_E1, MX23 to MACRO_F1, MX24 to MACRO_G1, MX25 to MACRO_H1, MX26 to MACRO_I1, MX20 to NUM_0, MX17 to NUM_1, MX11 to NUM_10, MX8 to NUM_2, MX18 to NUM_3, MX13 to NUM_4, MX14 to NUM_5, MX15 to NUM_6, MX9 to NUM_7, MX10 to NUM_8, MX12 to NUM_ADD1, MX6 to NUM_DIV1, MX21 to NUM_ENTER1, MX5 to NUM_LOCK1, MX27 to NUM_MULT1, MX19 to NUM_PERIOD1, MX7 to NUM_SUB1
Connections:
- net ROW2: now reaches D10.1 (K), D24.1 (K), D7.1 (K), D8.1 (K), D9.1 (K)
- net ROW3: now reaches D11.1 (K), D12.1 (K), D13.1 (K), D14.1 (K), D25.1 (K)
- net at D25.2 (A): now also MACRO_F1.2
- net COL4: now reaches MACRO_C1.1, NUM_10.1, NUM_3.1, NUM_6.1, NUM_MULT1.1, NUM_PERIOD1.1
- net COL2: now reaches MACRO_A1.1, NUM_0.1, NUM_1.1, NUM_4.1, NUM_7.1, NUM_LOCK1.1
- net COL1: now reaches MACRO_E1.1, MACRO_F1.1, MACRO_G1.1, MACRO_H1.1, MACRO_I1.1
- net at MACRO_H1.2: now also D27.2 (A)
- net COL5: now reaches MACRO_D1.1, NUM_ADD1.1, NUM_ENTER1.1, NUM_SUB1.1
- net at MACRO_G1.2: now also D26.2 (A)
- net at MACRO_I1.2: now also D28.2 (A)
- net ROW1: now reaches D3.1 (K), D4.1 (K), D5.1 (K), D6.1 (K)
- net ROW1: now also D29.1 (K)
- net ROW5: now reaches D18.1 (K), D19.1 (K), D20.1 (K), D21.1 (K), D27.1 (K)
- net ROW4: now reaches D15.1 (K), D16.1 (K), D17.1 (K), D26.1 (K)
- net COL3: now reaches MACRO_B1.1, NUM_2.1, NUM_5.1, NUM_8.1, NUM_DIV1.1
- net ROW6: now reaches D22.1 (K), D23.1 (K), D28.1 (K)
- net at D24.2 (A): now also MACRO_E1.2
- net ROT+: now reaches SW1.A
- net ROT-: now reaches SW1.B
- net ROT_VCC: now reaches SW1.C
- net at SW1.S: now also D29.2 (A)
Other:
- moved on the sheet: D10, D11, D12, D13, D14, D15, D16, D17, D18, D19, D20, D21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

Commit message: ROT_SW
Disconnect after S diode, ROT_SW
Connections:
- net ROW1: no longer D29.1 (K)
- new net ROT_SW: D29.1 (K)
Changed lines of the file:
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@@
-	)
-	(junction
-		(at 78.74 60.96)
-		(diameter 0)
-		(color 0 0 0 0)
 	)
 	(junction
@@
 	(wire
 		(pts
-			(xy 62.23 60.96) (xy 78.74 60.96)
-		)
-		(stroke
-			(width 0)
-			(type default)
-		)
-	)
-	(wire
-		(pts
 			(xy 43.18 149.86) (xy 48.26 149.86)
 		)
@@
 		)
 	)
+	(hierarchical_label "ROT_SW"
+		(shape input)
+		(at 62.23 60.96 270)
+		(effects
+			(font
+				(size 1.27 1.27)
+			)
+			(justify right)
+		)
+	)

Commit message: pcb stuff
Parts:
- added LED1, LED10, LED11, LED12, LED13, LED14, LED15, LED16, LED17, LED18, LED19, LED2, LED20, LED21, LED22, LED23, LED24, LED25, LED26, LED27, LED3, LED4, LED5, LED6, LED7, LED8, LED9: MX_SK6812MINI-E, PCM_marbastlib-mx:LED_MX_6028R, symbol PCM_marbastlib-mx:MX_SK6812MINI-E
- D10, D11, D12, D13, D14, D15, D16, D17, D18, D19, D20, D21, D22, D23, D24, D25, D26, D27, D28, D29, D3, D4, D5, D6, D7, D8, D9: value 1N4148 -> 1N4148W; footprint PCM_Diode_THT_AKL:D_DO-35_SOD27_P7.62mm_Horizontal -> PCM_Diode_SMD_AKL:D_SOD-123; symbol PCM_Diode_AKL:1N4148 -> PCM_Diode_AKL:1N4148W
Connections:
- new net: LED24.2 (DOUT), LED25.3 (DIN)
- new net: LED23.2 (DOUT), LED24.3 (DIN)
- new net: LED8.3 (DIN), LED9.2 (DOUT)
- new net: LED10.2 (DOUT), LED9.3 (DIN)
- new net: LED22.2 (DOUT), LED23.3 (DIN)
- new net: LED14.3 (DIN), LED15.2 (DOUT)
- new net: LED15.3 (DIN), LED6.2 (DOUT)
- new net: LED20.2 (DOUT), LED26.3 (DIN)
- new net: LED20.3 (DIN), LED27.2 (DOUT)
- new net: LED1.3 (DIN), LED2.2 (DOUT)
- new net: LED2.3 (DIN), LED3.2 (DOUT)
- new net: LED4.3 (DIN), LED5.2 (DOUT)
- new net: LED25.2 (DOUT), LED27.3 (DIN)
- new net: LED18.3 (DIN), LED19.2 (DOUT)
- new net: LED11.2 (DOUT), LED19.3 (DIN)
- new net: LED11.3 (DIN), LED12.2 (DOUT)
- new net: LED12.3 (DIN), LED13.2 (DOUT)
- new net: LED13.3 (DIN), LED14.2 (DOUT)
- new net: LED21.2 (DOUT), LED22.3 (DIN)
- new net: LED16.3 (DIN), LED17.2 (DOUT)
- new net: LED17.3 (DIN), LED18.2 (DOUT)
- new net: LED3.3 (DIN), LED4.2 (DOUT)
- new net: LED6.3 (DIN), LED7.2 (DOUT)
- new net: LED16.2 (DOUT), LED21.3 (DIN)
- new net: LED7.3 (DIN), LED8.2 (DOUT)
- new net: LED1.2 (DOUT), LED10.3 (DIN)
- new net DIN: LED5.3 (DIN)
- new net VDD: LED1.1 (VDD), LED10.1 (VDD), LED11.1 (VDD), LED12.1 (VDD), LED13.1 (VDD), LED14.1 (VDD), LED15.1 (VDD), LED16.1 (VDD), LED17.1 (VDD), LED18.1 (VDD), LED19.1 (VDD), LED2.1 (VDD), LED20.1 (VDD), LED21.1 (VDD), LED22.1 (VDD), LED23.1 (VDD), LED24.1 (VDD), LED25.1 (VDD), LED26.1 (VDD), LED27.1 (VDD), LED3.1 (VDD), LED4.1 (VDD), LED5.1 (VDD), LED6.1 (VDD), LED7.1 (VDD), LED8.1 (VDD), LED9.1 (VDD)
- new net VSS: LED1.4 (VSS), LED10.4 (VSS), LED11.4 (VSS), LED12.4 (VSS), LED13.4 (VSS), LED14.4 (VSS), LED15.4 (VSS), LED16.4 (VSS), LED17.4 (VSS), LED18.4 (VSS), LED19.4 (VSS), LED2.4 (VSS), LED20.4 (VSS), LED21.4 (VSS), LED22.4 (VSS), LED23.4 (VSS), LED24.4 (VSS), LED25.4 (VSS), LED26.4 (VSS), LED27.4 (VSS), LED3.4 (VSS), LED4.4 (VSS), LED5.4 (VSS), LED6.4 (VSS), LED7.4 (VSS), LED8.4 (VSS), LED9.4 (VSS)
Other:
- moved on the sheet: D10, D11, D12, D13, D14, D15, D16, D17, D18, D19, D20, D21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
