File: hardware/numpad/numpad/numpad.kicad_pcb (KiCad board)
At the start: 4 copper layers, 123.8 x 142.9 mm, 119 parts, among them IC1 LD1117-3.3V-SOT223, J1 Conn_01x06, SW1 ROT_SKYLOONG_HS, SW2 Push_Button, Y1 8MHz

Commit message: commit before merging to dev
Routing:
- net GND: track 7.92 -> 19.9 mm
Changed lines of the file:
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@@
+	)
+	(segment
+		(start 67.627 50.47)
+		(end 68.722 49.375)
+		(width 0.2)
+		(layer "B.Cu")
+		(net 1)
+	)
+	(segment
+		(start 58.543751 72.949999)
+		(end 65.550001 72.949999)
+		(width 0.2)
+		(layer "B.Cu")
+		(net 1)
 	)
 	(segment
 		(start 67.543751 78.343751)
 		(end 67.2 78)
+		(width 0.2)
+		(layer "B.Cu")
+		(net 1)
+	)
+	(segment
+		(start 61.177 50.47)
+		(end 60.082 49.375)
 		(width 0.2)
 		(layer "B.Cu")
@@
 		(width 0.2)
 		(layer "B.Cu")
+		(net 1)
+	)
+	(segment
+		(start 61.177 50.79)
+		(end 61.177 50.47)
+		(width 0.2)
+		(layer "B.Cu")
+		(net 1)
+	)
+	(segment
+		(start 65.550001 72.949999)
+		(end 66.4 72.1)
+		(width 0.2)
+		(layer "B.Cu")
+		(net 1)
+	)
+	(segment
+		(start 67.627 50.79)
+		(end 67.627 50.47)
+		(width 0.2)
+		(layer "B.Cu")
