File: hardware/68percent/68percent.kicad_pcb (KiCad board)
At the start: 4 copper layers, 176 parts, among them IC1 LD1117-3.3V-SOT223, J1 Conn_01x06, SW2 Push_Button, Y1 8MHz

Commit message: layout adjustment
Parts:
- removed S5: MX_stab, PCM_marbastlib-mx:STAB_MX_2u
- KEY_ALT1, KEY_CTRL1, KEY_SPACE1, KEY_WIN1: footprint PCM_marbastlib-mx:SW_MX_HS_CPG151101S11_1u -> PCM_Switch_Keyboard_Hotswap_Kailh:SW_Hotswap_Kailh_MX_Plated_1.25u; moved to F.Cu
- KEY_SHIFT2: footprint PCM_marbastlib-mx:SW_MX_HS_CPG151101S11_1u -> PCM_Switch_Keyboard_Hotswap_Kailh:SW_Hotswap_Kailh_MX_Plated_1.75u; moved to F.Cu
- KEY_\1: footprint PCM_marbastlib-mx:SW_MX_HS_CPG151101S11_1u -> PCM_marbastlib-mx:SW_MX_HS_CPG151101S11_1.5u
- S4: footprint PCM_marbastlib-mx:STAB_MX_2.25u -> PCM_marbastlib-mx:STAB_MX_P_2.25u
- moved KEY_ALT1 99.7 mm to (-23.8, 123.8), turned to 0 degrees
- moved KEY_PGDN1 85.7 mm to (259.6, 104.8)
- moved S3 72.9 mm to (231.0, 47.6)
- moved KEY_UARROW1 64.3 mm to (240.5, 104.8)
- moved KEY_DARROW1 63.3 mm to (221.5, 123.8)
- moved KEY_CAPS1 61.9 mm to (-19.1, 85.7)
- moved KEY_SHIFT2 61.6 mm to (214.3, 104.8), turned to 0 degrees
- moved KEY_0 59.6 mm to (164.3, 47.6)
- moved KEY_5 59.6 mm to (69.0, 47.6)
- moved KEY_T1 59.6 mm to (78.5, 66.7)
- moved KEY_Y1 59.6 mm to (97.6, 66.7)
- moved KEY_[1 59.6 mm to (192.9, 66.7)
- moved KEY_]1 59.6 mm to (211.9, 66.7)
- moved KEY_3 59.6 mm to (30.9, 47.6)
- moved KEY_4 59.6 mm to (50.0, 47.6)
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
Commit message: layout adjustment
Parts:
- moved KEY_ENTER1 104.2 mm to (323.5, 128.6)
- moved S4 104.2 mm to (323.5, 128.6)
- moved KEY_.1 104.2 mm to (264.0, 147.6)
- moved KEY_DARROW2 104.2 mm to (335.4, 166.7)
- moved KEY_UARROW1 104.2 mm to (335.4, 147.6)
- moved KEY_[1 104.2 mm to (287.8, 109.5)
- moved KEY_'1 104.2 mm to (292.6, 128.6)
- moved KEY_6 104.2 mm to (183.0, 90.5)
- moved KEY_;1 104.2 mm to (273.5, 128.6)
- moved KEY_A1 104.2 mm to (102.1, 128.6)
- moved KEY_D1 104.2 mm to (140.2, 128.6)
- moved KEY_G1 104.2 mm to (178.3, 128.6)
- moved KEY_J1 104.2 mm to (216.4, 128.6)
- moved KEY_K1 104.2 mm to (235.4, 128.6)
- moved KEY_L1 104.2 mm to (254.5, 128.6)
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Other:
- board outline added: 333.4 x 142.9 mm

Commit message: footprint
Parts:
- added LED1: choc_SK6812MINI-E, PCM_marbastlib-choc:LED_choc_6028R, B.Cu at (215.7, 2.02)
- added LED10: choc_SK6812MINI-E, PCM_marbastlib-choc:LED_choc_6028R, B.Cu at (215.7, 47.5)
- added LED11: choc_SK6812MINI-E, PCM_marbastlib-choc:LED_choc_6028R, B.Cu at (215.7, 52.5)
- added LED12: choc_SK6812MINI-E, PCM_marbastlib-choc:LED_choc_6028R, B.Cu at (215.7, 57.6)
- added LED13: choc_SK6812MINI-E, PCM_marbastlib-choc:LED_choc_6028R, B.Cu at (206.9, 2.02)
- added LED14: choc_SK6812MINI-E, PCM_marbastlib-choc:LED_choc_6028R, B.Cu at (206.9, 7.08)
- added LED15: choc_SK6812MINI-E, PCM_marbastlib-choc:LED_choc_6028R, B.Cu at (206.9, 12.1)
- added LED16: choc_SK6812MINI-E, PCM_marbastlib-choc:LED_choc_6028R, B.Cu at (206.9, 17.2)
- added LED17: choc_SK6812MINI-E, PCM_marbastlib-choc:LED_choc_6028R, B.Cu at (206.9, 22.2)
- added LED18: choc_SK6812MINI-E, PCM_marbastlib-choc:LED_choc_6028R, B.Cu at (206.9, 27.3)
- added LED19: choc_SK6812MINI-E, PCM_marbastlib-choc:LED_choc_6028R, B.Cu at (206.9, 32.3)
- added LED2: choc_SK6812MINI-E, PCM_marbastlib-choc:LED_choc_6028R, B.Cu at (215.7, 7.08)
- added LED20: choc_SK6812MINI-E, PCM_marbastlib-choc:LED_choc_6028R, B.Cu at (206.9, 37.4)
- added LED21: choc_SK6812MINI-E, PCM_marbastlib-choc:LED_choc_6028R, B.Cu at (206.9, 42.4)
- added LED22: choc_SK6812MINI-E, PCM_marbastlib-choc:LED_choc_6028R, B.Cu at (206.9, 47.5)
- added LED23: choc_SK6812MINI-E, PCM_marbastlib-choc:LED_choc_6028R, B.Cu at (206.9, 52.5)
- added LED24: choc_SK6812MINI-E, PCM_marbastlib-choc:LED_choc_6028R, B.Cu at (206.9, 57.6)
- added LED25: choc_SK6812MINI-E, PCM_marbastlib-choc:LED_choc_6028R, B.Cu at (198.0, 2.02)
- added LED26: choc_SK6812MINI-E, PCM_marbastlib-choc:LED_choc_6028R, B.Cu at (198.0, 7.08)
- added LED27: choc_SK6812MINI-E, PCM_marbastlib-choc:LED_choc_6028R, B.Cu at (198.0, 12.1)
- added LED28: choc_SK6812MINI-E, PCM_marbastlib-choc:LED_choc_6028R, B.Cu at (198.0, 17.2)
- added LED29: choc_SK6812MINI-E, PCM_marbastlib-choc:LED_choc_6028R, B.Cu at (198.0, 22.2)
- added LED3: choc_SK6812MINI-E, PCM_marbastlib-choc:LED_choc_6028R, B.Cu at (215.7, 12.1)
- added LED30: choc_SK6812MINI-E, PCM_marbastlib-choc:LED_choc_6028R, B.Cu at (198.0, 27.3)
- added LED31: choc_SK6812MINI-E, PCM_marbastlib-choc:LED_choc_6028R, B.Cu at (198.0, 32.3)
- added LED32: choc_SK6812MINI-E, PCM_marbastlib-choc:LED_choc_6028R, B.Cu at (198.0, 37.4)
- added LED33: choc_SK6812MINI-E, PCM_marbastlib-choc:LED_choc_6028R, B.Cu at (198.0, 42.4)
- added LED34: choc_SK6812MINI-E, PCM_marbastlib-choc:LED_choc_6028R, B.Cu at (198.0, 47.5)
- added LED35: choc_SK6812MINI-E, PCM_marbastlib-choc:LED_choc_6028R, B.Cu at (198.0, 52.5)
- added LED36: choc_SK6812MINI-E, PCM_marbastlib-choc:LED_choc_6028R, B.Cu at (198.0, 57.6)
- added LED37: choc_SK6812MINI-E, PCM_marbastlib-choc:LED_choc_6028R, B.Cu at (189.1, 2.02)
- added LED38: choc_SK6812MINI-E, PCM_marbastlib-choc:LED_choc_6028R, B.Cu at (189.1, 7.08)
- added LED39: choc_SK6812MINI-E, PCM_marbastlib-choc:LED_choc_6028R, B.Cu at (189.1, 12.1)
- added LED4: choc_SK6812MINI-E, PCM_marbastlib-choc:LED_choc_6028R, B.Cu at (215.7, 17.2)
- added LED40: choc_SK6812MINI-E, PCM_marbastlib-choc:LED_choc_6028R, B.Cu at (189.1, 17.2)
- added LED41: choc_SK6812MINI-E, PCM_marbastlib-choc:LED_choc_6028R, B.Cu at (189.1, 22.2)
- added LED42: choc_SK6812MINI-E, PCM_marbastlib-choc:LED_choc_6028R, B.Cu at (189.1, 27.3)
- added LED43: choc_SK6812MINI-E, PCM_marbastlib-choc:LED_choc_6028R, B.Cu at (189.1, 32.3)
- added LED44: choc_SK6812MINI-E, PCM_marbastlib-choc:LED_choc_6028R, B.Cu at (189.1, 37.4)
- added LED45: choc_SK6812MINI-E, PCM_marbastlib-choc:LED_choc_6028R, B.Cu at (189.1, 42.4)
- added LED46: choc_SK6812MINI-E, PCM_marbastlib-choc:LED_choc_6028R, B.Cu at (189.1, 47.5)
- added LED47: choc_SK6812MINI-E, PCM_marbastlib-choc:LED_choc_6028R, B.Cu at (189.1, 52.5)
- added LED48: choc_SK6812MINI-E, PCM_marbastlib-choc:LED_choc_6028R, B.Cu at (189.1, 57.6)
- added LED49: choc_SK6812MINI-E, PCM_marbastlib-choc:LED_choc_6028R, B.Cu at (180.3, 2.02)
- added LED5: choc_SK6812MINI-E, PCM_marbastlib-choc:LED_choc_6028R, B.Cu at (215.7, 22.2)
- added LED50: choc_SK6812MINI-E, PCM_marbastlib-choc:LED_choc_6028R, B.Cu at (180.3, 7.08)
- added LED51: choc_SK6812MINI-E, PCM_marbastlib-choc:LED_choc_6028R, B.Cu at (180.3, 12.1)
- added LED52: choc_SK6812MINI-E, PCM_marbastlib-choc:LED_choc_6028R, B.Cu at (180.3, 17.2)
- added LED53: choc_SK6812MINI-E, PCM_marbastlib-choc:LED_choc_6028R, B.Cu at (180.3, 22.2)
- added LED54: choc_SK6812MINI-E, PCM_marbastlib-choc:LED_choc_6028R, B.Cu at (180.3, 27.3)
- added LED55: choc_SK6812MINI-E, PCM_marbastlib-choc:LED_choc_6028R, B.Cu at (180.3, 32.3)
- added LED56: choc_SK6812MINI-E, PCM_marbastlib-choc:LED_choc_6028R, B.Cu at (180.3, 37.4)
- added LED57: choc_SK6812MINI-E, PCM_marbastlib-choc:LED_choc_6028R, B.Cu at (180.3, 42.4)
- added LED58: choc_SK6812MINI-E, PCM_marbastlib-choc:LED_choc_6028R, B.Cu at (180.3, 47.5)
- added LED59: choc_SK6812MINI-E, PCM_marbastlib-choc:LED_choc_6028R, B.Cu at (180.3, 52.5)
- added LED6: choc_SK6812MINI-E, PCM_marbastlib-choc:LED_choc_6028R, B.Cu at (215.7, 27.3)
- added LED60: choc_SK6812MINI-E, PCM_marbastlib-choc:LED_choc_6028R, B.Cu at (180.3, 57.6)
- added LED61: choc_SK6812MINI-E, PCM_marbastlib-choc:LED_choc_6028R, B.Cu at (171.4, 2.02)
- added LED62: choc_SK6812MINI-E, PCM_marbastlib-choc:LED_choc_6028R, B.Cu at (171.4, 7.08)
- added LED63: choc_SK6812MINI-E, PCM_marbastlib-choc:LED_choc_6028R, B.Cu at (171.4, 12.1)
- added LED64: choc_SK6812MINI-E, PCM_marbastlib-choc:LED_choc_6028R, B.Cu at (171.4, 17.2)
- added LED65: choc_SK6812MINI-E, PCM_marbastlib-choc:LED_choc_6028R, B.Cu at (171.4, 22.2)
- added LED66: choc_SK6812MINI-E, PCM_marbastlib-choc:LED_choc_6028R, B.Cu at (171.4, 27.3)
- added LED67: choc_SK6812MINI-E, PCM_marbastlib-choc:LED_choc_6028R, B.Cu at (171.4, 32.3)
- added LED68: choc_SK6812MINI-E, PCM_marbastlib-choc:LED_choc_6028R, B.Cu at (171.4, 37.4)
- added LED7: choc_SK6812MINI-E, PCM_marbastlib-choc:LED_choc_6028R, B.Cu at (215.7, 32.3)
- added LED8: choc_SK6812MINI-E, PCM_marbastlib-choc:LED_choc_6028R, B.Cu at (215.7, 37.4)
- added LED9: choc_SK6812MINI-E, PCM_marbastlib-choc:LED_choc_6028R, B.Cu at (215.7, 42.4)
- added S5: MX_stab, PCM_marbastlib-mx:STAB_MX_P_2u, F.Cu at (181.5, 71.6)
Connections:
- U1 pad 20: /ROT_SW -> unconnected-(U1-PA4-Pad20)
- U1 pad 22: /ROT_TIMB -> unconnected-(U1-PA6-Pad22)
- U1 pad 23: /ROT_TIMA -> unconnected-(U1-PA7-Pad23)

Commit message: LEDs
Parts:
- moved LED68 226.7 mm to (354.2, 171.5), turned to 0 degrees
- moved LED67 215.1 mm to (335.4, 171.5), turned to 0 degrees
- moved LED66 204.5 mm to (316.4, 171.5), turned to 0 degrees
- moved LED58 203.3 mm to (354.5, 152.2), turned to 0 degrees
- moved LED65 195.3 mm to (297.3, 171.5), turned to 0 degrees
- moved LED44 191.1 mm to (354.5, 133.2), turned to 0 degrees
- moved LED57 190.0 mm to (335.2, 152.4), turned to 0 degrees
- moved LED64 187.5 mm to (278.0, 171.5), turned to 0 degrees
- moved LED63 181.8 mm to (259.0, 171.5), turned to 0 degrees
- moved LED30 179.0 mm to (354.5, 114.1), turned to 0 degrees
- moved LED61 177.3 mm to (118.7, 171.3), turned to 0 degrees
- moved LED1 174.1 mm to (68.6, 95.1), turned to 0 degrees
- moved LED56 172.6 mm to (309.0, 152.4), turned to 0 degrees
- moved LED15 169.3 mm to (354.5, 95.1), turned to 0 degrees
- moved LED43 168.0 mm to (323.5, 133.2), turned to 0 degrees
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
Commit message: diode placement
Parts:
- C1, C10, C11, C2, C3, C4, C5, C6, C7, C8, C9, D1, D2, East1, FB1, IC1, North1, R1, R10, R13, R2, R3, R4, R5, R6, R7, R8, R9, SW2, South1, U1, West1, Y1: moved to F.Cu
- D10, D11, D12, D13, D14, D15, D16, D17, D18, D19, D20, D21, D22, D23, D24, D25, D26, D27, D28, D29, D3, D30, D31, D32, D33, D34, D35, D36, D37, D38, D39, D4, D40, D41, D42, D43, D44, D45, D46, D47, D48, D5, D50, D51, D52, D53, D54, D55, D56, D57, D58, D59, D6, D60, D61, D62, D64, D65, D68, D7, D71, D72, D73, D74, D75, D76, D8, D9: footprint PCM_Diode_SMD_AKL:D_SOD-123 -> PCM_Diode_THT_AKL:D_DO-35_SOD27_P7.62mm_Horizontal; moved to F.Cu
- moved D64 526.6 mm to (303.9, 64.1), turned to -90 degrees
- moved D18 525.9 mm to (326.5, 64.1), turned to -90 degrees
- moved D3 523.6 mm to (328.9, 64.1), turned to -90 degrees
- moved D19 523.4 mm to (324.1, 64.1), turned to -90 degrees
- moved D50 523.3 mm to (306.3, 64.1), turned to -90 degrees
- moved D20 520.9 mm to (321.8, 64.1), turned to -90 degrees
- moved D36 520.3 mm to (308.7, 64.1), turned to -90 degrees
- moved D65 518.6 mm to (288.4, 64.1), turned to -90 degrees
- moved D21 518.4 mm to (319.4, 64.1), turned to -90 degrees
- moved D22 510.0 mm to (311.0, 64.1), turned to -90 degrees
- moved D4 507.8 mm to (313.4, 64.1), turned to -90 degrees
- moved D51 507.7 mm to (290.8, 64.1), turned to -90 degrees
- moved D37 504.6 mm to (293.2, 64.1), turned to -90 degrees
- moved D23 502.1 mm to (295.6, 64.1), turned to -90 degrees
- moved D52 492.1 mm to (275.3, 64.1), turned to -90 degrees
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Routing:
- net /ROW4: track 0.00 -> 280.0 mm, vias 0 -> 14
- net /ROW5: track 0.00 -> 269.1 mm, vias 0 -> 10
- net /ROW3: track 0.00 -> 263.4 mm, vias 0 -> 14
- net /ROW2: track 0.00 -> 250.0 mm, vias 0 -> 15
- net /ROW1: track 0.00 -> 232.2 mm, vias 0 -> 15
- net Net-(D5-A): track 0.00 -> 19.6 mm, vias 0 -> 2
- net Net-(D13-A): track 0.00 -> 19.6 mm, vias 0 -> 2
- net Net-(D14-A): track 0.00 -> 19.6 mm, vias 0 -> 2
- net Net-(D4-A): track 0.00 -> 19.6 mm, vias 0 -> 2
- net Net-(D9-A): track 0.00 -> 19.1 mm, vias 0 -> 2
- net Net-(D7-A): track 0.00 -> 19.1 mm, vias 0 -> 2
- net Net-(D30-A): track 0.00 -> 19.1 mm, vias 0 -> 2
- net Net-(D26-A): track 0.00 -> 19.1 mm, vias 0 -> 2
- net Net-(D22-A): track 0.00 -> 19.1 mm, vias 0 -> 2
- net Net-(D18-A): track 0.00 -> 19.1 mm, vias 0 -> 2
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Other:
- board size 333.4 x 142.9 mm -> 319.1 x 142.9 mm

Commit message: pushy
Parts:
- D10, D11, D12, D13, D14, D15, D16, D17, D22, D23, D24, D25, D26, D27, D28, D29, D30, D31, D32, D33, D34, D35, D36, D37, D38, D39, D4, D40, D41, D42, D43, D44, D45, D46, D47, D48, D5, D50, D51, D52, D53, D54, D55, D56, D57, D58, D59, D6, D60, D61, D62, D64, D65, D68, D7, D71, D72, D73, D74, D75, D76, D8, D9: moved to B.Cu
- moved C1 252.2 mm to (114.5, 59.4), turned to 90 degrees
- moved C11 249.7 mm to (114.5, 68.1), turned to 90 degrees
- moved FB1 245.8 mm to (101.0, 68.1)
- moved C6 242.7 mm to (93.4, 57.6), turned to 90 degrees
- moved C2 241.8 mm to (101.0, 59.5), turned to 90 degrees
- moved C5 235.4 mm to (98.7, 78.0), turned to -90 degrees
- moved C9 230.6 mm to (89.9, 57.6), turned to -90 degrees
- moved C3 230.1 mm to (95.9, 78.0), turned to -90 degrees
- moved C10 229.7 mm to (86.8, 57.6), turned to 90 degrees
- moved C4 221.3 mm to (84.4, 77.9), turned to -90 degrees
- moved D2 211.3 mm to (55.7, 61.9), turned to 90 degrees
- moved D76 211.2 mm to (330.6, 64.1)
- moved D3 207.9 mm to (121.1, 64.1)
- moved D62 206.5 mm to (328.2, 64.1)
- moved D18 203.1 mm to (123.4, 64.1)
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Routing:
- net Net-(J1-Pin_6): track 0.00 -> 239.5 mm
- net Net-(J1-Pin_5): track 0.00 -> 236.7 mm
- net Net-(J1-Pin_4): track 0.00 -> 233.9 mm
- net Net-(J1-Pin_2): track 0.00 -> 228.6 mm
- net Net-(D7-A): track 19.1 -> 2.64 mm, vias 2 -> 0
- net Net-(D22-A): track 19.1 -> 2.64 mm, vias 2 -> 0
- net Net-(D18-A): track 19.1 -> 2.64 mm, vias 2 -> 0
- net Net-(D9-A): track 19.1 -> 2.64 mm, vias 2 -> 0
- net Net-(D30-A): track 19.1 -> 2.64 mm, vias 2 -> 0
- net Net-(D26-A): track 19.1 -> 2.64 mm, vias 2 -> 0
- net Net-(D11-A): track 19.1 -> 2.64 mm, vias 2 -> 0
- net Net-(D10-A): track 19.1 -> 2.64 mm, vias 2 -> 0
- net Net-(D35-A): track 19.1 -> 2.64 mm, vias 2 -> 0
- net Net-(D32-A): track 19.1 -> 2.64 mm, vias 2 -> 0
- net Net-(D16-A): track 19.1 -> 2.64 mm, vias 2 -> 0
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
Commit message: traces
Routing:
- net Net-(D3-A): track 3.37 -> 66.0 mm
- net Net-(D4-A): track 3.37 -> 63.1 mm
- net Net-(D5-A): track 3.37 -> 62.1 mm
- net Net-(D6-A): track 2.64 -> 55.0 mm
- net Net-(D17-A): track 3.37 -> 51.2 mm
- net Net-(D7-A): track 2.64 -> 49.7 mm
- net Net-(D8-A): track 3.37 -> 46.2 mm
- net Net-(D9-A): track 2.64 -> 41.6 mm
- net Net-(D10-A): track 2.64 -> 39.3 mm
- net Net-(D13-A): track 3.37 -> 39.4 mm, vias 0 -> 2
- net Net-(D16-A): track 2.64 -> 36.4 mm
- net Net-(D14-A): track 3.37 -> 34.6 mm
- net Net-(D11-A): track 2.64 -> 33.7 mm
- net Net-(D12-A): track 3.37 -> 28.2 mm
- net Net-(D15-A): track 2.64 -> 24.0 mm
