File: hardware/68percent/68percent.kicad_pcb (KiCad board)
At the start: 4 copper layers, 319.1 x 142.9 mm, 244 parts, among them IC1 LD1117-3.3V-SOT223, J1 Conn_01x06, SW2 Push_Button, Y1 8MHz

Commit message: traces
Routing:
- net /COL3: track 0.00 -> 148.6 mm, vias 0 -> 4
- net /COL1: track 0.00 -> 117.5 mm
- net /COL2: track 0.00 -> 100.7 mm, vias 0 -> 2
- net /COL9: track 0.00 -> 67.0 mm
- net /COL7: track 0.00 -> 67.0 mm
- net /COL6: track 0.00 -> 67.0 mm
- net /COL5: track 0.00 -> 67.0 mm
- net /COL4: track 0.00 -> 67.0 mm
- net /COL8: track 0.00 -> 67.0 mm
- net Net-(D22-A): track 2.64 -> 68.6 mm, vias 0 -> 2

Commit message: Traces
67676767676767
SIX SEVEN
Routing:
- net /COL12: track 0.00 -> 100.3 mm
- net /COL13: track 0.00 -> 96.6 mm
- net /COL11: track 0.00 -> 90.2 mm
- net /COL10: track 0.00 -> 89.5 mm
- net /COL15: track 0.00 -> 76.2 mm
- net /COL14: track 0.00 -> 66.7 mm
- net Net-(D3-A): track 66.0 -> 128.9 mm
- net Net-(J1-Pin_4): track 233.9 -> 283.7 mm, vias 0 -> 2
- net Net-(J1-Pin_2): track 228.6 -> 265.3 mm, vias 0 -> 4
- net Net-(J1-Pin_6): track 239.5 -> 274.4 mm
- net Net-(J1-Pin_5): track 236.7 -> 259.0 mm
- net /NRST: track 0.00 -> 7.25 mm
- net +3.3V: track 0.00 -> 4.23 mm
- net Net-(U1-BOOT): track 0.00 -> 3.75 mm

Commit message: traces
676767676767
Routing:
- net Net-(D19-A): track 0.00 -> 104.3 mm, vias 0 -> 6
- net Net-(D18-A): track 2.64 -> 80.0 mm, vias 0 -> 4
- net Net-(D3-A): track 128.9 -> 62.2 mm
- net Net-(D21-A): track 3.37 -> 0.00 mm
- net Net-(D20-A): track 2.64 -> 0.00 mm

Commit message: traces
six seven
Routing:
- net Net-(D20-A): track 0.00 -> 130.1 mm, vias 0 -> 2
- net Net-(D21-A): track 0.00 -> 119.0 mm, vias 0 -> 6
- net Net-(D36-A): track 9.29 -> 0.00 mm
- net Net-(D4-A): track 63.1 -> 59.8 mm
- net Net-(D64-A): track 3.37 -> 0.00 mm
- net Net-(D50-A): track 2.64 -> 0.00 mm
- net Net-(D22-A): track 68.6 -> 66.0 mm

Commit message: traces
Routing:
- net Net-(D64-A): track 0.00 -> 130.2 mm, vias 0 -> 12
- net Net-(D50-A): track 0.00 -> 104.7 mm, vias 0 -> 6
- net Net-(D51-A): track 2.64 -> 104.1 mm, vias 0 -> 6
- net Net-(D36-A): track 0.00 -> 85.7 mm, vias 0 -> 8
- net Net-(D37-A): track 9.29 -> 83.5 mm, vias 0 -> 6
- net Net-(D23-A): track 2.64 -> 67.3 mm, vias 0 -> 4
- net Net-(D5-A): track 62.1 -> 58.7 mm
- net Net-(D65-A): track 3.37 -> 0.00 mm
