File: hardware/68percent/68percent.kicad_sch (KiCad schematic)
At the start: 35 parts, among them IC1 LD1117-3.3V-SOT223, J1 Conn_01x06, SW2 Push_Button, Y1 8MHz

Commit message: somebody once told me the world is gonna roll me
Connections:
- net ROT_SW: no longer names the net of U1.20 (PA4)
- net ROT_TIMA: no longer names the net of U1.23 (PA7)
- net ROT_TIMB: no longer names the net of U1.22 (PA6)
Other:
- added sheet RGB Lights (untitled.kicad_sch)
Changed lines of the file:
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@@
 	(wire
 		(pts
-			(xy 162.56 132.08) (xy 162.56 151.13)
-		)
-		(stroke
-			(width 0)
-			(type default)
-		)
-	)
-	(wire
-		(pts
 			(xy 147.32 77.47) (xy 147.32 88.9)
 		)
@@
 	(wire
 		(pts
-			(xy 154.94 132.08) (xy 154.94 147.32)
-		)
-		(stroke
-			(width 0)
-			(type default)
-		)
-	)
-	(wire
-		(pts
 			(xy 119.38 129.54) (xy 113.03 129.54)
 		)
@@
 	(wire
 		(pts
-			(xy 160.02 132.08) (xy 160.02 151.13)
-		)
-		(stroke
-			(width 0)
-			(type default)
-		)
-	)
-	(wire
-		(pts
 			(xy 170.18 74.93) (xy 170.18 88.9)
 		)
@@
 		)
 	)
-	(label "ROT_TIMA"
-		(at 162.56 151.13 90)
-		(effects
-			(font
-				(size 1.27 1.27)
-			)
-			(justify left bottom)
-		)
-	)
 	(label "COL3"
 		(at 237.49 26.67 270)
@@
 		)
 	)
+	(label "RGB_DATAIN"
+		(at 237.49 113.03 180)
+		(effects
+			(font
+				(size 1.27 1.27)
+			)
+			(justify right bottom)
+		)
+	)
 	(label "UART_RX_WEST"
 		(at 212.09 106.68 180)
@@
 		)
 	)
-	(label "ROT_SW"
-		(at 154.94 147.32 90)
-		(effects
-			(font
-				(size 1.27 1.27)
-			)
-			(justify left bottom)
-		)
-	)
 	(label "UART_RX_SOUTH"
 		(at 53.34 92.71 0)
@@
 		)
 	)
-	(label "ROT_TIMB"
-		(at 160.02 151.13 90)
-		(effects
-			(font
-				(size 1.27 1.27)
-			)
-			(justify left bottom)
-		)
-	)
 	(symbol
 		(lib_id "PCM_4ms_Power-symbol:GND")
@@
 				)
 			)
+		)
+	)
+	(sheet
+		(at 241.3 93.98)
+		(size 36.83 20.32)
+		(exclude_from_sim no)
+		(in_bom yes)
+		(on_board yes)
+		(dnp no)
+		(fields_autoplaced yes)
+		(stroke
+			(width 0.1524)
+			(type solid)
+		)
+		(fill
+			(color 0 0 0 0.0000)
+		)
+		(property "Sheetname" "RGB Lights"
+			(at 241.3 93.2684 0)
+			(effects
+				(font
+					(size 1.27 1.27)
+				)
+				(justify left bottom)
+			)
+		)
+		(property "Sheetfile" "untitled.kicad_sch"
+			(at 241.3 114.8846 0)
+			(effects
+				(font
+					(size 1.27 1.27)
+				)
+				(justify left top)
+			)
+		)
+		(instances
+			(project "68percent"
+				(path "/a3d0d559-cac8-4859-ad0f-79ad0c1a1a82"
+					(page "3")
+				)
+			)

Commit message: traces
Other:
- sheet RGB Lights ports: added RGB IN; removed none
Changed lines of the file:
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@@
 	(wire
 		(pts
+			(xy 237.49 111.76) (xy 237.49 113.03)
+		)
+		(stroke
+			(width 0)
+			(type default)
+		)
+	)
+	(wire
+		(pts
 			(xy 43.18 58.42) (xy 49.53 58.42)
 		)
@@
 	(wire
 		(pts
+			(xy 241.3 111.76) (xy 237.49 111.76)
+		)
+		(stroke
+			(width 0)
+			(type default)
+		)
+	)
+	(wire
+		(pts
 			(xy 222.25 101.6) (xy 231.14 101.6)
 		)
@@
 			)
 		)
+		(pin "RGB IN" input
+			(at 241.3 111.76 180)
+			(effects
+				(font
+					(size 1.27 1.27)
+				)
+				(justify left)
+			)
+		)

Commit message: pcb update
Connections:
- net COL1: now also U1.34 (PB13); no longer U1.59 (PB7)
- net COL10: now also U1.51 (PA10); no longer U1.39 (PC8)
- net COL11: now also U1.52 (PC11); no longer U1.38 (PC7)
- net COL12: now also U1.56 (PB4); no longer U1.37 (PC6)
- net COL13: now also U1.57 (PB5); no longer U1.36 (PB15)
- net COL14: now also U1.58 (PB6); no longer U1.35 (PB14)
- net COL15: now also U1.59 (PB7); no longer U1.34 (PB13)
- net COL2: now also U1.35 (PB14); no longer U1.58 (PB6)
- net COL3: now also U1.36 (PB15); no longer U1.57 (PB5)
- net COL4: now also U1.37 (PC6); no longer U1.56 (PB4)
- net COL5: now also U1.38 (PC7); no longer U1.52 (PC11)
- net COL6: now also U1.39 (PC8); no longer U1.51 (PA10)
- net COL7: now also U1.40 (PC9); no longer U1.50 (PA15)
- net COL9: now also U1.50 (PA15); no longer U1.40 (PC9)
- net UART_RX_NORTH: now also U1.17 (PA3); no longer U1.54 (PD2)
- net UART_RX_SOUTH: now also U1.54 (PD2); no longer U1.17 (PA3)
- net UART_TX_NORTH: now also U1.16 (PA2); no longer U1.53 (PC12)
- net UART_TX_SOUTH: now also U1.53 (PC12); no longer U1.16 (PA2)
